File: circuits/miniv_motor_controller_board/miniv_motor_controller_board/miniv_motor_controller_board.kicad_pcb (KiCad board)
At the start: 2 copper layers, 78 x 102 mm, 4 parts

Commit message: update board
Signed-off-by: Masaya Kataoka <ms.kataoka@gmail.com>
Parts:
- added C1: 0.1u, Capacitor_THT:C_Disc_D5.1mm_W3.2mm_P5.00mm, F.Cu at (106.0, 126.0)
- added D2: LED, LED_THT:LED_D3.0mm, F.Cu at (104.0, 104.5)
- added F1: Fuse, 3557-15:3557-15, F.Cu at (65.0, 55.0)
- added J1: DC_in, Connector_AMASS:AMASS_XT60PW-F_1x02_P7.20mm_Horizontal, F.Cu at (107.0, 58.0)
- added J2: T200_ESC_power, Connector_AMASS:AMASS_XT60PW-F_1x02_P7.20mm_Horizontal, F.Cu at (89.0, 58.0)
- added J3: T200_ESC_signal, Connector_AMASS:AMASS_XT30PW-F_1x02_P2.50mm_Horizontal, F.Cu at (69.0, 141.0)
- added J4: Conn_EStop_Signal, Connector_JST:JST_XH_B2B-XH-A_1x02_P2.50mm_Vertical, F.Cu at (90.0, 65.0)
- added JP2: Relay_NO, Connector_Wire:SolderWire-0.5sqmm_1x01_D0.9mm_OD2.1mm, F.Cu at (58.0, 61.0)
- added JP4: Relay_SIG, Connector_Wire:SolderWire-0.1sqmm_1x01_D0.4mm_OD1mm, F.Cu at (54.0, 105.0)
- added JP5: Relay_GND, Connector_Wire:SolderWire-0.1sqmm_1x01_D0.4mm_OD1mm, F.Cu at (45.0, 105.0)
- added JP6: Relay_VCC, Connector_Wire:SolderWire-0.1sqmm_1x01_D0.4mm_OD1mm, F.Cu at (108.0, 71.0)
- added JP7: Relay_COM, Connector_Wire:SolderWire-0.5sqmm_1x01_D0.9mm_OD2.1mm, F.Cu at (100.0, 68.0)
- added M78AR05-1: ~, M78AR05-1:M78AR05-1, F.Cu at (112.0, 66.0)
- added Q1: 2SC1815, Package_TO_SOT_THT:TO-92_Inline, F.Cu at (100.0, 83.0)
- added Q2: 2SC1815, Package_TO_SOT_THT:TO-92_Inline, F.Cu at (100.0, 90.0)
- added R1: 100k, Resistor_THT:R_Axial_DIN0207_L6.3mm_D2.5mm_P10.16mm_Horizontal, F.Cu at (105.0, 86.0)
- added R2: 100k, Resistor_THT:R_Axial_DIN0207_L6.3mm_D2.5mm_P10.16mm_Horizontal, F.Cu at (105.0, 92.5)
- added R4: 470, Resistor_THT:R_Axial_DIN0207_L6.3mm_D2.5mm_P10.16mm_Horizontal, F.Cu at (84.0, 83.0)
- added R5: 390, Resistor_THT:R_Axial_DIN0207_L6.3mm_D2.5mm_P10.16mm_Horizontal, F.Cu at (58.0, 85.0)
- added R6: 1K, Resistor_THT:R_Axial_DIN0207_L6.3mm_D2.5mm_P10.16mm_Horizontal, F.Cu at (58.0, 97.5)
- added R7: 1K, Resistor_THT:R_Axial_DIN0207_L6.3mm_D2.5mm_P10.16mm_Horizontal, F.Cu at (63.5, 97.5)
- added R8: 390, Resistor_THT:R_Axial_DIN0207_L6.3mm_D2.5mm_P10.16mm_Horizontal, F.Cu at (63.5, 85.0)
- added SW1: SW_isolation, SS-12D00G3:SS-12D00G3, F.Cu at (65.0, 130.0)
- added SW2: SW_disable_EStop, SS-12D00G3:SS-12D00G3, F.Cu at (112.0, 102.0)
- added U1: Teensy4.1, Teensy_Custom:Teensy41, F.Cu at (89.0, 115.0)
- added U2: TLP624, Package_DIP:DIP-4_W7.62mm, F.Cu at (50.0, 80.0)
- added U3: TLP624, Package_DIP:DIP-4_W7.62mm, F.Cu at (108.0, 77.0)
- added U4: ~, AE-RELAY953B-12V:AE-RELAY953B-12V, F.Cu at (70.0, 86.0)
- added U5: ~, RJLD-260YC1:RJLD-260YC1, F.Cu at (101.0, 139.0)
- moved H4 21.3 mm to (118.0, 146.0)
- moved H3 20.5 mm to (118.0, 54.0)
- moved H1 19.4 mm to (46.0, 146.0)
- moved H2 18.6 mm to (46.0, 54.0)
Routing:
- net GND: track 0.00 -> 248.8 mm
- net Net-(M78AR05-1-Vout): track 0.00 -> 114.3 mm
- net Net-(J3-Pin_2): track 0.00 -> 90.2 mm
- net Net-(JP4-A): track 0.00 -> 71.2 mm
- net Net-(R7-Pad1): track 0.00 -> 53.0 mm
- net Net-(U5-GND): track 0.00 -> 51.1 mm
- net Net-(U1-LED): track 0.00 -> 44.4 mm
- net Net-(SW1-C): track 0.00 -> 34.4 mm
- net Net-(J4-Pin_1): track 0.00 -> 28.9 mm
- net Net-(J4-Pin_2): track 0.00 -> 28.1 mm
- net Net-(D2-A): track 0.00 -> 27.9 mm
- net +12V: track 0.00 -> 27.7 mm
- net Net-(U1-T+): track 0.00 -> 27.2 mm
- net Net-(U1-T-): track 0.00 -> 25.2 mm
- net Net-(U1-R+): track 0.00 -> 23.7 mm
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Other:
- board size 78 x 102 mm -> 80 x 100 mm

Commit message: modify circuit
Signed-off-by: Masaya Kataoka <ms.kataoka@gmail.com>
Parts:
- removed Q1, Q2: 2SC1815, Package_TO_SOT_THT:TO-92_Inline
- added U6: ~, Package_DIP:DIP-14_W7.62mm, F.Cu at (149.1, 105.4)
- R1, R2: value 100k -> 1k
- R4: value 470 -> 390
- SW1: value SW_isolation -> SW_Push_DPDT; footprint SS-12D00G3:SS-12D00G3 -> 2MD1-T2-B4-M2-Q-N:2MD1-T2-B4-M2-Q-N
- moved SW1 100.4 mm to (155.5, 86.5), turned to 0 degrees
- moved R4 50.0 mm to (132.8, 72.5)
Connections:
- J3 pad 1: GND -> Net-(J3-Pin_1)
- R6 pad 1: Net-(SW1-C) -> Net-(R6-Pad1)
- SW1 pad 1: Net-(J3-Pin_2) -> Net-(SW1-A-Pad1)
- SW1 pad 2: Net-(SW1-B) -> Net-(J3-Pin_1)
- SW1 pad 3: Net-(SW1-C) -> GND
- U1 pad 33: Net-(SW1-B) -> unconnected-(U1-41_A17-Pad33)
- U2 pad 3: GND -> Net-(SW1-A-Pad1)
- U2 pad 4: Net-(J3-Pin_2) -> Net-(SW1-A-Pad4)
Routing:
- net Net-(J3-Pin_2): track 90.2 -> 0.00 mm
- net Net-(JP4-A): track 71.2 -> 0.00 mm
- net Net-(M78AR05-1-Vout): track 114.3 -> 65.9 mm
- net Net-(SW1-C): track 34.4 -> 0.00 mm
- net Net-(D2-A): track 27.9 -> 0.00 mm
- net GND: track 248.8 -> 224.7 mm
- net Net-(SW1-B): track 18.2 -> 0.00 mm
- net Net-(U6-1A): track 5.02 -> 0.06 mm
- net Net-(U6-1B): track 5.19 -> 0.65 mm

Commit message: re-design board
Signed-off-by: Masaya Kataoka <ms.kataoka@gmail.com>
Parts:
- added U7: ~, MIWI06-24S12:MIWI06-24S12, F.Cu at (80.0, 78.5)
- moved U6 101.6 mm to (47.5, 107.0)
- moved SW1 87.1 mm to (80.0, 130.0)
- moved R4 78.1 mm to (60.5, 102.0), turned to 180 degrees
- moved JP5 73.0 mm to (118.0, 102.5)
- moved U2 64.6 mm to (74.0, 140.0), turned to 0 degrees
- moved R5 59.8 mm to (68.0, 144.0)
- moved JP6 57.8 mm to (50.5, 65.5)
- moved R1 56.4 mm to (49.0, 92.6), turned to 90 degrees
- moved U3 56.3 mm to (52.0, 71.5), turned to -90 degrees
- moved R2 54.7 mm to (50.5, 97.0)
- moved M78AR05-1 53.8 mm to (59.0, 75.5), turned to -90 degrees
- moved SW2 44.8 mm to (67.5, 97.0), turned to 0 degrees
- moved R6 30.4 mm to (63.0, 127.5), turned to -90 degrees
- moved J4 28.8 mm to (114.0, 81.0), turned to -90 degrees
- moved D2 24.6 mm to (79.5, 102.0), turned to 180 degrees
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Connections:
- D2 pad 1: GND -> GNDREF
- J1 pad 1: GND -> GNDREF_Bat
- J1 pad 2: +12V -> Net-(J1-Pin_2)
- J2 pad 1: GND -> GNDREF_Bat
- JP5 pad 1: GND -> GNDREF
- JP7 pad 1: +12V -> Net-(J1-Pin_2)
- M78AR05-1 pad 2: GND -> GNDREF
- R6 pad 1: Net-(R6-Pad1) -> Net-(U1-41_A17)
- SW1 pad 3: GND -> Net-(SW1-C-Pad3)
- SW1 pad 4: Net-(SW1-A-Pad4) -> Net-(U1-41_A17)
- SW1 pad 6: Net-(R6-Pad1) -> Net-(SW1-C-Pad6)
- SW2 pad 1: GND -> GNDREF
- U1 pad 1: GND -> GNDREF
- U1 pad 33: unconnected-(U1-41_A17-Pad33) -> Net-(U1-41_A17)
- U1 pad 34: GND -> Net-(SW1-A-Pad1)
- U2 pad 2: GND -> Net-(SW1-A-Pad1)
- U2 pad 3: Net-(SW1-A-Pad1) -> Net-(SW1-C-Pad3)
- U2 pad 4: Net-(SW1-A-Pad4) -> Net-(SW1-C-Pad6)
- U6 pad 7: GND -> GNDREF
Routing:
- net GND: track 224.7 -> 0.00 mm
- net GNDREF: track 0.00 -> 145.8 mm
- net Net-(M78AR05-1-Vout): track 65.9 -> 131.6 mm
- net Net-(J4-Pin_1): track 28.9 -> 83.8 mm
- net GNDREF_Bat: track 0.00 -> 50.6 mm
- net Net-(SW1-A-Pad1): track 0.00 -> 41.1 mm
- net Net-(J3-Pin_1): track 0.00 -> 34.4 mm
- net Net-(R7-Pad1): track 53.0 -> 24.6 mm
- net Net-(J3-Pin_2): track 0.00 -> 27.3 mm
- net Net-(U1-41_A17): track 0.00 -> 20.4 mm
- net Net-(U6-1B): track 0.65 -> 20.8 mm
- net Net-(J1-Pin_2): track 0.00 -> 19.1 mm
- net Net-(D2-A): track 0.00 -> 16.5 mm
- net Net-(JP4-A): track 0.00 -> 14.8 mm
- net Net-(SW1-C-Pad3): track 0.00 -> 11.3 mm
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