File: circuits/miniv_motor_controller_board/miniv_motor_controller_board/miniv_motor_controller_board.kicad_pcb (KiCad board)
At the start: 2 copper layers, 80 x 100 mm, 33 parts, among them J1 DC_in, J2 T200_ESC_power, J3 T200_ESC_signal, J4 Conn_EStop_Signal, SW1 SW_Push_DPDT, SW2 SW_disable_EStop, U1 Teensy4.1, U2 TLP624, U3 TLP624

Commit message: remove R1/R2
Signed-off-by: Masaya Kataoka <ms.kataoka@gmail.com>
Parts:
- removed R1, R2: 1k, Resistor_THT:R_Axial_DIN0207_L6.3mm_D2.5mm_P10.16mm_Horizontal
Connections:
- U3 pad 3: Net-(R1-Pad2) -> Net-(U6-1B)
- U6 pad 1: Net-(U6-1A) -> Net-(SW2-B)
Routing:
- net Net-(SW2-B): track 8.08 -> 29.8 mm
- net Net-(U6-1B): track 20.8 -> 34.4 mm
- net Net-(U6-1A): track 11.2 -> 0.00 mm
- net Net-(R1-Pad2): track 3.49 -> 0.00 mm
