File: circuits/miniv_motor_controller_board/miniv_motor_controller_board/miniv_motor_controller_board.kicad_pcb (KiCad board)
At the start: 2 copper layers, 80 x 100 mm, 31 parts, among them J1 DC_in, J2 T200_ESC_power, J3 T200_ESC_signal, J4 Conn_EStop_Signal, SW1 SW_Push_DPDT, SW2 SW_disable_EStop, U1 Teensy4.1, U2 TLP624, U3 TLP624

Commit message: add R1/R2
Signed-off-by: Masaya Kataoka <ms.kataoka@gmail.com>
Parts:
- added R1: 1K, Resistor_THT:R_Axial_DIN0207_L6.3mm_D2.5mm_P10.16mm_Horizontal, F.Cu at (60.5, 97.0)
- added R2: 1K, Resistor_THT:R_Axial_DIN0207_L6.3mm_D2.5mm_P10.16mm_Horizontal, F.Cu at (49.0, 83.0)
Connections:
- U3 pad 3: Net-(U6-1B) -> Net-(R2-Pad1)
- U6 pad 1: Net-(SW2-B) -> Net-(U6-1A)
Routing:
- net Net-(SW2-B): track 29.8 -> 8.24 mm
- net Net-(U6-1B): track 34.4 -> 19.8 mm
- net Net-(U6-1A): track 0.00 -> 11.2 mm
- net Net-(R2-Pad1): track 0.00 -> 4.07 mm

Commit message: add solid pattern to the board
Signed-off-by: Masaya Kataoka <ms.kataoka@gmail.com>
Routing:
- added copper zone on B.Cu, net GNDREF
- added copper zone on F.Cu, net GNDREF
Changed lines of the file:
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@@
 		(net 97)
 	)
+	(zone
+		(net 92)
+		(net_name "GNDREF")
+		(layers "F&B.Cu")
+		(hatch edge 0.5)
+		(connect_pads
+			(clearance 0.5)
+		)
+		(min_thickness 0.25)
+		(filled_areas_thickness no)
+		(fill yes
+			(thermal_gap 0.5)
+			(thermal_bridge_width 0.5)
+		)
+		(polygon
+			(pts
+				(xy 42 50) (xy 122 50) (xy 122 108.5) (xy 42 108.5)
+			)
+		)
+	)
+	(zone
+		(net 92)
+		(net_name "GNDREF")
+		(layers "F&B.Cu")
+		(hatch edge 0.5)
+		(priority 1)
+		(connect_pads
+			(clearance 0.5)
+		)
+		(min_thickness 0.25)
+		(filled_areas_thickness no)
+		(fill yes
+			(thermal_gap 0.5)
+			(thermal_bridge_width 0.5)
+		)
+		(polygon
+			(pts
+				(xy 87.5 150) (xy 87.5 108.5) (xy 42 108.5) (xy 42 150)
+			)
+		)
+	)
 )
