File: circuits/miniv_motor_controller_board/miniv_motor_controller_board/miniv_motor_controller_board.kicad_sch (KiCad schematic)
At the start: 33 parts, among them J1 DC_in, J2 T200_ESC_power, J3 T200_ESC_signal, J4 Conn_EStop_Signal, SW1 SW_Push_DPDT, SW2 SW_disable_EStop, U1 Teensy4.1, U2 TLP624, U3 TLP624

Commit message: add datasheet field
Signed-off-by: Masaya Kataoka <ms.kataoka@gmail.com>
Connections:
- net at U4. (VCC(CN1-1)): now also JP2.2 (B)
Changed lines of the file:
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@@
 			)
 		)
-		(property "Datasheet" "~"
+		(property "Datasheet" "https://akizukidenshi.com/catalog/g/g118155/"
 			(at 281.94 67.31 0)
 			(effects
@@
 			)
 		)
-		(property "Datasheet" "~"
+		(property "Datasheet" "https://akizukidenshi.com/catalog/g/g115707/"
 			(at 147.32 88.9 0)
 			(effects
@@
 			)
 		)
-		(property "Datasheet" ""
+		(property "Datasheet" "https://akizukidenshi.com/catalog/g/g106533/"
 			(at 217.17 49.53 0)
 			(effects
@@
 			)
 		)
-		(property "Datasheet" ""
+		(property "Datasheet" "https://akizukidenshi.com/catalog/g/g106095/"
 			(at 219.71 128.27 0)
 			(effects
@@
 			)
 		)
-		(property "Datasheet" "~"
+		(property "Datasheet" "https://akizukidenshi.com/catalog/g/g118155/"
 			(at 281.94 90.17 0)
 			(effects
@@
 			)
 		)
-		(property "Datasheet" "~"
+		(property "Datasheet" "https://akizukidenshi.com/catalog/g/g118223/"
 			(at 269.24 87.63 0)
 			(effects
@@
 			)
 		)
-		(property "Datasheet" "~"
+		(property "Datasheet" "https://akizukidenshi.com/catalog/g/g112247/"
 			(at 114.3 161.29 0)
 			(effects
@@
 			)
 		)
-		(property "Datasheet" ""
+		(property "Datasheet" "https://www.digikey.jp/ja/products/detail/sparkfun-electronics/DEV-20359/16688101"
 			(at 39.37 109.22 0)
 			(effects
@@
 			)
 		)
-		(property "Datasheet" ""
+		(property "Datasheet" "https://akizukidenshi.com/catalog/g/g113536/"
 			(at 158.75 77.47 0)
 			(effects
@@
 			)
 		)
-		(property "Datasheet" "~"
+		(property "Datasheet" "https://akizukidenshi.com/catalog/g/g100301/"
 			(at 107.95 97.79 0)
 			(effects

Commit message: add XT30 to the board
Signed-off-by: Masaya Kataoka <ms.kataoka@gmail.com>
Connections:
- net at U4. (VCC(CN1-1)): now also JP2.2 (B)
Changed lines of the file:
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@@
 			)
 		)
-		(property "Datasheet" "~"
+		(property "Datasheet" "https://akizukidenshi.com/catalog/g/g117948"
 			(at 118.11 96.52 0)
 			(effects

Commit message: fix: ERC error
Connections:
- net at JP5.2 (B): now also U4.2 (GND(CN1-2)); no longer U4. (VCC(CN1-1))
- net at JP7.2 (B): now also U4.4 (COM(CN2-1)); no longer U4. (VCC(CN1-1))
- net at JP6.2 (B): now also U4.1 (VCC(CN1-1)); no longer U4. (VCC(CN1-1))
- net at JP4.2 (B): now also U4.3 (SIG(CN1-3)); no longer U4. (VCC(CN1-1))
- net at JP2.2 (B): now also U4.5 (NO(CN2-2)); no longer U4. (VCC(CN1-1))
Changed lines of the file:
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@@
 (kicad_sch
-	(version 20231120)
+	(version 20250114)
 	(generator "eeschema")
-	(generator_version "8.0")
+	(generator_version "9.0")
 	(paper "A4")
 	(junction
@@
 			)
 		)
-		(pin ""
+		(pin "3"
 		)
-		(pin ""
+		(pin "6"
 		)
-		(pin ""
+		(pin "5"
 		)
-		(pin ""
+		(pin "2"
 		)
-		(pin ""
+		(pin "1"
 		)
-		(pin ""
+		(pin "4"
 		)
 		(instances
@@
 		)
 	)
+	(embedded_fonts no)
 )
