File: circuits/miniv_estop_board/miniv_estop_board/miniv_estop_board.kicad_sch (KiCad schematic)
At the start: 39 parts, among them J1 Conn_Main_DCDC, J2 Conn_neopixel_01, J3 Conn_neopixel_02, J4 Conn_neopixel_03, J5 Conn_neopixel_04, J6 EStop_button, J7 EStop_signal0, J8 EStop_signal1, Q1 2SJ555-E, Q2 NPN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

Commit message: update mkdocs.yaml
Signed-off-by: Masaya Kataoka <ms.kataoka@gmail.com>
Connections:
- net GND: now also J1.1 (Pin_1), J2.1 (Pin_1), J3.1 (Pin_1), J4.1 (Pin_1), J5.1 (Pin_1), Q1.1 (G), Q6.1 (G), R1.2, R16.1, R2.1, U1.47 (GND)
Changed lines of the file:
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@@
 	)
 	(junction
+		(at 44.45 38.1)
+		(diameter 0)
+		(color 0 0 0 0)
+	)
+	(junction
 		(at 234.95 39.37)
 		(diameter 0)
@@
 	(wire
 		(pts
-			(xy 36.83 38.1) (xy 54.61 38.1)
+			(xy 36.83 38.1) (xy 44.45 38.1)
 		)
 		(stroke
@@
 	(wire
 		(pts
+			(xy 44.45 38.1) (xy 54.61 38.1)
+		)
+		(stroke
+			(width 0)
+			(type default)
+		)
+	)
+	(wire
+		(pts
 			(xy 92.71 59.69) (xy 234.95 59.69)
 		)
@@
 					(unit 1)
 				)
+			)
+		)
+	)
+	(symbol
+		(lib_id "power:GND")
+		(at 44.45 38.1 0)
+		(unit 1)
+		(exclude_from_sim no)
+		(in_bom yes)
+		(on_board yes)
+		(dnp no)
+		(fields_autoplaced yes)
+		(property "Reference" "#PWR01"
+			(at 44.45 44.45 0)
+			(effects
+				(font
+					(size 1.27 1.27)
+				)
+				(hide yes)
+			)
+		)
+		(property "Value" "GND"
+			(at 44.45 43.18 0)
+			(effects
+				(font
+					(size 1.27 1.27)
+				)
+			)
+		)
+		(property "Footprint" ""
+			(at 44.45 38.1 0)
+			(effects
+				(font
+					(size 1.27 1.27)
+				)
+				(hide yes)
+			)
+		)
+		(property "Datasheet" ""
+			(at 44.45 38.1 0)
+			(effects
+				(font
+					(size 1.27 1.27)
+				)
+				(hide yes)
+			)
+		)
+		(property "Description" "Power symbol creates a global label with name \"GND\" , ground"
+			(at 44.45 38.1 0)
+			(effects
+				(font
+					(size 1.27 1.27)
+				)
+				(hide yes)
+			)
+		)
+		(pin "1"
+		)
+		(instances
+			(project ""
+				(path "/1034f469-1e36-4dd4-a538-1c7038a139d6"
+					(reference "#PWR01")
+					(unit 1)
+				)

Commit message: modify connection
Signed-off-by: Masaya Kataoka <ms.kataoka@gmail.com>
Connections:
- net at D1.2 (A), J2.3 (Pin_3), J3.3 (Pin_3)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: no longer R10.1, R9.1
- net at D3.2 (A), J4.3 (Pin_3), J5.3 (Pin_3)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: now also R10.1, R9.1
Changed lines of the file:
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@@
-	)
-	(junction
-		(at 195.58 44.45)
-		(diameter 0)
-		(color 0 0 0 0)
 	)
 	(junction
@@
 	)
 	(junction
-		(at 210.82 44.45)
-		(diameter 0)
-		(color 0 0 0 0)
-	)
-	(junction
 		(at 93.98 110.49)
 		(diameter 0)
@@
 	)
 	(junction
+		(at 195.58 64.77)
+		(diameter 0)
+		(color 0 0 0 0)
+	)
+	(junction
 		(at 39.37 30.48)
 		(diameter 0)
@@
 	)
 	(junction
+		(at 210.82 64.77)
+		(diameter 0)
+		(color 0 0 0 0)
+	)
+	(junction
 		(at 54.61 38.1)
 		(diameter 0)
@@
 	(wire
 		(pts
-			(xy 210.82 44.45) (xy 232.41 44.45)
-		)
-		(stroke
-			(width 0)
-			(type default)
-		)
-	)
-	(wire
-		(pts
 			(xy 238.76 54.61) (xy 232.41 54.61)
 		)
@@
 	(wire
 		(pts
+			(xy 210.82 64.77) (xy 210.82 71.12)
+		)
+		(stroke
+			(width 0)
+			(type default)
+		)
+	)
+	(wire
+		(pts
 			(xy 130.81 87.63) (xy 130.81 91.44)
 		)
@@
 	(wire
 		(pts
-			(xy 195.58 44.45) (xy 195.58 71.12)
-		)
-		(stroke
-			(width 0)
-			(type default)
-		)
-	)
-	(wire
-		(pts
 			(xy 180.34 78.74) (xy 180.34 81.28)
 		)
@@
 	(wire
 		(pts
-			(xy 149.86 64.77) (xy 232.41 64.77)
+			(xy 149.86 64.77) (xy 195.58 64.77)
 		)
 		(stroke
@@
 	(wire
 		(pts
+			(xy 195.58 64.77) (xy 195.58 71.12)
+		)
+		(stroke
+			(width 0)
+			(type default)
+		)
+	)
+	(wire
+		(pts
 			(xy 39.37 52.07) (xy 50.8 52.07)
 		)
@@
 	(wire
 		(pts
+			(xy 195.58 64.77) (xy 210.82 64.77)
+		)
+		(stroke
+			(width 0)
+			(type default)
+		)
+	)
+	(wire
+		(pts
 			(xy 238.76 74.93) (xy 232.41 74.93)
 		)
@@
 	(wire
 		(pts
-			(xy 210.82 44.45) (xy 210.82 71.12)
-		)
-		(stroke
-			(width 0)
-			(type default)
-		)
-	)
-	(wire
-		(pts
 			(xy 195.58 78.74) (xy 195.58 81.28)
 		)
@@
 	(wire
 		(pts
+			(xy 210.82 64.77) (xy 232.41 64.77)
+		)
+		(stroke
+			(width 0)
+			(type default)
+		)
+	)
+	(wire
+		(pts
 			(xy 39.37 30.48) (xy 39.37 52.07)
 		)
@@
 	(wire
 		(pts
-			(xy 195.58 44.45) (xy 210.82 44.45)
+			(xy 180.34 44.45) (xy 232.41 44.45)
 		)
 		(stroke
@@
 		)
 		(stroke
-			(width 0)
-			(type default)
-		)
-	)
-	(wire
-		(pts
-			(xy 180.34 44.45) (xy 195.58 44.45)
-		)
-		(stroke

Commit message: Feature/add capaciter regester for neopixel (#383)
* add capaciter

Signed-off-by: Masaya Kataoka <ms.kataoka@gmail.com>

* update bom

Signed-off-by: Masaya Kataoka <ms.kataoka@gmail.com>

* update pcb

Signed-off-by: Masaya Kataoka <ms.kataoka@gmail.com>

---------

Signed-off-by: Masaya Kataoka <ms.kataoka@gmail.com>
Parts:
- added C2, C6, C7, C9: 1000μ, Capacitor_THT:CP_Radial_D12.5mm_P5.00mm, symbol Device:C_Polarized
- added R12, R13, R14, R15: 470, R_Axial_DIN0207_L6.3mm_D2.5mm_P10.16mm_Horizontal, symbol Device:R
Connections:
- net GND: now also C2.2, C6.2, C7.2, C9.2
- net at Q7.2 (C), R4.2: now also R12.2; no longer J2.2 (Pin_2)
- net at Q2.2 (C), R8.2: now also R13.2; no longer J3.2 (Pin_2)
- net at D3.2 (A), J4.3 (Pin_3), J5.3 (Pin_3)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: now also C7.1, C9.1
- net at Q4.2 (C), R10.2: now also R15.2; no longer J5.2 (Pin_2)
- net at Q3.2 (C), R9.2: now also R14.2; no longer J4.2 (Pin_2)
- net at D1.2 (A), J2.3 (Pin_3), J3.3 (Pin_3)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: now also C2.1, C6.1
- new net: J4.2 (Pin_2), R14.1
- new net: J2.2 (Pin_2), R12.1
- new net: J3.2 (Pin_2), R13.1
- new net: J5.2 (Pin_2), R15.1
